File: schematics/kill-switch-remote/kill-switch.sch (KiCad schematic (older format))
At the start: 14 parts, among them SW1 MB, SW2 RB, SW3 LB, U1 NRF24L01_Breakout

Commit message: Fixed switch error
Parts:
- renumbered R4 to R2, R2 to R3, R3 to R4, SW3 to SW1, SW1 to SW2, SW2 to SW3
Connections:
- wire segments 61 -> 63
Other:
- note added: "C1 is placed across transciver vcc and gnd.\nC2 and C3 are placed across arduino +5V and gnd.\nLB - Left Button\nMB- Middle Button\nRB - Right Button\nthis is with the arduino usb port pointed to the right.\nPush left button to activate D4.\nPush middle button to activate d3.\nPush right button to activate D2.\n"
- note removed: "C1 is placed across transciver vcc and gnd.\nC2 and C3 are placed across arduino +5V and gnd.\nLB - Left Button\nMB- Middle Button\nRB - Right Button\nthis is with the arduino usb port pointed to the right.\nPush left button to activate D4.\nPush middle button to activate d3.\nPush middle and right button to activate D2 and D3.\n"
Changed lines of the file:
@@
 	8150 3750 8150 3650
 $Comp
-L Switch:SW_Push SW1
+L Switch:SW_Push SW2
 U 1 1 5C491E40
 P 5800 3300
-F 0 "SW1" V 5850 3500 50  0000 R CNN
+F 0 "SW2" V 5850 3500 50  0000 R CNN
 F 1 "MB" V 5750 3500 50  0000 R CNN
 F 2 "" H 5800 3500 50  0001 C CNN
@@
 L Device:R_US R1
 U 1 1 5C49209B
-P 6300 4750
-F 0 "R1" V 6095 4750 50  0000 C CNN
-F 1 "220" V 6186 4750 50  0000 C CNN
-F 2 "" V 6340 4740 50  0001 C CNN
-F 3 "~" H 6300 4750 50  0001 C CNN
-	1    6300 4750
+P 6300 4850
+F 0 "R1" V 6095 4850 50  0000 C CNN
+F 1 "220" V 6186 4850 50  0000 C CNN
+F 2 "" V 6340 4840 50  0001 C CNN
+F 3 "~" H 6300 4850 50  0001 C CNN
+	1    6300 4850
 	0    1    1    0
 $EndComp
@@
 	5300 4950 5300 4900
 $Comp
-L Device:R_US R2
+L Device:R_US R3
 U 1 1 5C4920CD
-P 5800 3900
-F 0 "R2" H 5732 3854 50  0000 R CNN
-F 1 "10k" H 5732 3945 50  0000 R CNN
-F 2 "" V 5840 3890 50  0001 C CNN
-F 3 "~" H 5800 3900 50  0001 C CNN
-	1    5800 3900
+P 5800 3750
+F 0 "R3" H 5732 3704 50  0000 R CNN
+F 1 "10k" H 5732 3795 50  0000 R CNN
+F 2 "" V 5840 3740 50  0001 C CNN
+F 3 "~" H 5800 3750 50  0001 C CNN
+	1    5800 3750
 	1    0    0    1
 $EndComp
@@
 L power:GND #PWR?
 U 1 1 5C5447B7
-P 5800 4100
-F 0 "#PWR?" H 5800 3850 50  0001 C CNN
-F 1 "GND" H 5805 3927 50  0000 C CNN
-F 2 "" H 5800 4100 50  0001 C CNN
-F 3 "" H 5800 4100 50  0001 C CNN
-	1    5800 4100
-	1    0    0    -1
-$EndComp
-Wire Wire Line
-	5800 4100 5800 4050
+P 5800 3950
+F 0 "#PWR?" H 5800 3700 50  0001 C CNN
+F 1 "GND" H 5805 3777 50  0000 C CNN
+F 2 "" H 5800 3950 50  0001 C CNN
+F 3 "" H 5800 3950 50  0001 C CNN
+	1    5800 3950
+	1    0    0    -1
+$EndComp
+Wire Wire Line
+	5800 3950 5800 3900
 $Comp
 L power:VCC #PWR?
@@
 	5800 5250 7550 5250
 $Comp
-L Switch:SW_Push SW3
+L Switch:SW_Push SW1
 U 1 1 5C550621
-P 7050 3300
-F 0 "SW3" V 7100 3500 50  0000 R CNN
-F 1 "LB" V 7000 3500 50  0000 R CNN
-F 2 "" H 7050 3500 50  0001 C CNN
-F 3 "" H 7050 3500 50  0001 C CNN
-	1    7050 3300
+P 5350 3300
+F 0 "SW1" V 5400 3500 50  0000 R CNN
+F 1 "LB" V 5300 3500 50  0000 R CNN
+F 2 "" H 5350 3500 50  0001 C CNN
+F 3 "" H 5350 3500 50  0001 C CNN
+	1    5350 3300
 	0    -1   -1   0
 $EndComp
 $Comp
-L Device:R_US R4
+L Device:R_US R2
 U 1 1 5C550628
-P 7050 3900
-F 0 "R4" H 6982 3854 50  0000 R CNN
-F 1 "10k" H 6982 3945 50  0000 R CNN
-F 2 "" V 7090 3890 50  0001 C CNN
-F 3 "~" H 7050 3900 50  0001 C CNN
-	1    7050 3900
+P 5350 3750
+F 0 "R2" H 5282 3704 50  0000 R CNN
+F 1 "10k" H 5282 3795 50  0000 R CNN
+F 2 "" V 5390 3740 50  0001 C CNN
+F 3 "~" H 5350 3750 50  0001 C CNN
+	1    5350 3750
 	1    0    0    1
 $EndComp
@@
 L power:GND #PWR?
 U 1 1 5C55062F
-P 7050 4100
-F 0 "#PWR?" H 7050 3850 50  0001 C CNN
-F 1 "GND" H 7055 3927 50  0000 C CNN
-F 2 "" H 7050 4100 50  0001 C CNN
-F 3 "" H 7050 4100 50  0001 C CNN
-	1    7050 4100
-	1    0    0    -1
-$EndComp
-Wire Wire Line
-	7050 4100 7050 4050
+P 5350 3950
+F 0 "#PWR?" H 5350 3700 50  0001 C CNN
+F 1 "GND" H 5355 3777 50  0000 C CNN
+F 2 "" H 5350 3950 50  0001 C CNN
+F 3 "" H 5350 3950 50  0001 C CNN
+	1    5350 3950
+	1    0    0    -1
+$EndComp
+Wire Wire Line
+	5350 3950 5350 3900
 $Comp
 L power:VCC #PWR?
 U 1 1 5C550636
-P 7050 3050
-F 0 "#PWR?" H 7050 2900 50  0001 C CNN
-F 1 "VCC" H 7067 3223 50  0000 C CNN
-F 2 "" H 7050 3050 50  0001 C CNN
-F 3 "" H 7050 3050 50  0001 C CNN
-	1    7050 3050
-	1    0    0    -1
-$EndComp
-Wire Wire Line
-	7050 3100 7050 3050
-$Comp
-L Switch:SW_Push SW2
+P 5350 3050
+F 0 "#PWR?" H 5350 2900 50  0001 C CNN
+F 1 "VCC" H 5367 3223 50  0000 C CNN
+F 2 "" H 5350 3050 50  0001 C CNN
+F 3 "" H 5350 3050 50  0001 C CNN
+	1    5350 3050
+	1    0    0    -1
+$EndComp
+Wire Wire Line
+	5350 3100 5350 3050
+$Comp
+L Switch:SW_Push SW3
 U 1 1 5C5569DB
-P 6100 3650
-F 0 "SW2" H 6300 3800 50  0000 R CNN
-F 1 "RB" H 6050 3800 50  0000 R CNN
-F 2 "" H 6100 3850 50  0001 C CNN
-F 3 "" H 6100 3850 50  0001 C CNN
-	1    6100 3650
-	1    0    0    -1
-$EndComp
-$Comp
-L Device:R_US R3
+P 6250 3300
+F 0 "SW3" V 6300 3500 50  0000 R CNN
+F 1 "RB" V 6200 3500 50  0000 R CNN
+F 2 "" H 6250 3500 50  0001 C CNN
+F 3 "" H 6250 3500 50  0001 C CNN
+	1    6250 3300
+	0    -1   -1   0
+$EndComp
+$Comp
+L Device:R_US R4
 U 1 1 5C5569E2
-P 6350 3900
-F 0 "R3" H 6282 3854 50  0000 R CNN
-F 1 "10k" H 6282 3945 50  0000 R CNN
-F 2 "" V 6390 3890 50  0001 C CNN
-F 3 "~" H 6350 3900 50  0001 C CNN
-	1    6350 3900
+P 6250 3750
+F 0 "R4" H 6182 3704 50  0000 R CNN
+F 1 "10k" H 6182 3795 50  0000 R CNN
+F 2 "" V 6290 3740 50  0001 C CNN
+F 3 "~" H 6250 3750 50  0001 C CNN
+	1    6250 3750
 	1    0    0    1
 $EndComp
@@
 L power:GND #PWR?
 U 1 1 5C5569E9
-P 6350 4100
-F 0 "#PWR?" H 6350 3850 50  0001 C CNN
-F 1 "GND" H 6355 3927 50  0000 C CNN
-F 2 "" H 6350 4100 50  0001 C CNN
-F 3 "" H 6350 4100 50  0001 C CNN
-	1    6350 4100
+P 6250 3950
+F 0 "#PWR?" H 6250 3700 50  0001 C CNN
+F 1 "GND" H 6255 3777 50  0000 C CNN
+F 2 "" H 6250 3950 50  0001 C CNN
+F 3 "" H 6250 3950 50  0001 C CNN
+	1    6250 3950
 	1    0    0    -1
 $EndComp
@@
 L Device:LED_Dual_AAC D1
 U 1 1 5C503668
-P 6850 4750
-F 0 "D1" H 7200 4450 50  0000 C CNN
-F 1 "LED_Dual_AAC" H 6850 4450 50  0000 C CNN
-F 2 "" H 6850 4750 50  0001 C CNN
-F 3 "~" H 6850 4750 50  0001 C CNN
-	1    6850 4750
+P 6850 4850
+F 0 "D1" H 7200 4550 50  0000 C CNN
+F 1 "LED_Dual_AAC" H 6850 4550 50  0000 C CNN
+F 2 "" H 6850 4850 50  0001 C CNN
+F 3 "~" H 6850 4850 50  0001 C CNN
+	1    6850 4850
 	1    0    0    -1
 $EndComp
@@
 L power:GND #PWR?
 U 1 1 5C509E9B
-P 6050 4850
-F 0 "#PWR?" H 6050 4600 50  0001 C CNN
-F 1 "GND" H 6055 4677 50  0000 C CNN
-F 2 "" H 6050 4850 50  0001 C CNN
-F 3 "" H 6050 4850 50  0001 C CNN
-	1    6050 4850
-	1    0    0    -1
-$EndComp
-Wire Wire Line
-	7150 4650 7550 4650
-Wire Wire Line
-	7150 4850 7200 4850
-Wire Wire Line
-	7200 4850 7200 4750
-Wire Wire Line
-	7200 4750 7550 4750
-Wire Wire Line
-	6450 4750 6550 4750
-Wire Wire Line
-	6050 4850 6050 4750
-Wire Wire Line
-	6050 4750 6150 4750
-Wire Wire Line
-	5800 3500 5800 3650
-Connection ~ 5800 3650
-Wire Wire Line
-	5800 3650 5800 3750
-Wire Wire Line
-	7050 3500 7050 3600
-Wire Wire Line
-	7550 4550 7250 4550
-Wire Wire Line
-	7250 4550 7250 3600
-Wire Wire Line
-	7250 3600 7050 3600
-Connection ~ 7050 3600
-Wire Wire Line
-	7050 3600 7050 3750
-Wire Wire Line
-	5550 3650 5550 4450
-Wire Wire Line
-	5550 3650 5800 3650
-Wire Wire Line
-	5550 4450 7550 4450
-Wire Wire Line
-	5900 3650 5800 3650
-Wire Wire Line
-	6350 4100 6350 4050
-Wire Wire Line
-	6350 3750 6350 3650
-Wire Wire Line
-	6350 3650 6300 3650
-Wire Wire Line
-	6350 3650 6550 3650
-Wire Wire Line
-	6550 3650 6550 4350
-Wire Wire Line
-	6550 4350 7550 4350
-Connection ~ 6350 3650
+P 6050 4950
+F 0 "#PWR?" H 6050 4700 50  0001 C CNN
+F 1 "GND" H 6055 4777 50  0000 C CNN
+F 2 "" H 6050 4950 50  0001 C CNN
+F 3 "" H 6050 4950 50  0001 C CNN
+	1    6050 4950
+	1    0    0    -1
+$EndComp
+Wire Wire Line
+	7300 4750 7550 4750
+Wire Wire Line
+	6050 4950 6050 4850
+Wire Wire Line
+	6050 4850 6150 4850
+Wire Wire Line
+	6250 3950 6250 3900
 Text Notes 9000 6400 0    50   ~ 0
-C1 is placed across transciver vcc and gnd.\nC2 and C3 are placed across arduino +5V and gnd.\nLB - Left Button\nMB- Middle Button\nRB - Right Button\nthis is with the arduino usb port pointed to the right.\nPush left button to activate D4.\nPush middle button to activate d3.\nPush middle and right button to activate D2 and D3.\n
+C1 is placed across transciver vcc and gnd.\nC2 and C3 are placed across arduino +5V and gnd.\nLB - Left Button\nMB- Middle Button\nRB - Right Button\nthis is with the arduino usb port pointed to the right.\nPush left button to activate D4.\nPush middle button to activate d3.\nPush right button to activate D2.\n
+$Comp
+L power:VCC #PWR?
+U 1 1 5C4FA7F3
+P 6250 3050
+F 0 "#PWR?" H 6250 2900 50  0001 C CNN
+F 1 "VCC" H 6267 3223 50  0000 C CNN
+F 2 "" H 6250 3050 50  0001 C CNN
+F 3 "" H 6250 3050 50  0001 C CNN
+	1    6250 3050
+	1    0    0    -1
+$EndComp
+Wire Wire Line
+	6250 3100 6250 3050
+Wire Wire Line
+	5550 3550 5350 3550
+Wire Wire Line
+	5350 3550 5350 3600
+Wire Wire Line
+	5350 3500 5350 3550
+Connection ~ 5350 3550
+Wire Wire Line
+	5800 3500 5800 3550
+Wire Wire Line
+	6250 3500 6250 3550
+Wire Wire Line
+	5800 3550 6000 3550
+Wire Wire Line
+	6000 3550 6000 4450
+Connection ~ 5800 3550
+Wire Wire Line
+	5800 3550 5800 3600
+Wire Wire Line
+	6000 4450 7550 4450
+Wire Wire Line
+	5550 4550 7550 4550
+Wire Wire Line
+	5550 3550 5550 4550
+Wire Wire Line
+	6250 3550 6450 3550
+Wire Wire Line
+	6450 3550 6450 4350
+Wire Wire Line
+	6450 4350 7550 4350
+Connection ~ 6250 3550
+Wire Wire Line
+	6250 3550 6250 3600
+Wire Wire Line
+	6450 4850 6550 4850
+Wire Wire Line
+	7300 4950 7150 4950
+Wire Wire Line
+	7300 4750 7300 4950
+Wire Wire Line
+	7250 4750 7250 4650
+Wire Wire Line
+	7250 4650 7550 4650
+Wire Wire Line
+	7150 4750 7250 4750
 $EndSCHEMATC
