File: schematics/kill-switch/kill-switch.sch (KiCad schematic (older format))
At the start: 14 parts, among them SW1 LB, SW2 MB, SW3 RB, U1 NRF24L01_Breakout

Commit message: motor/servo schematic finished. Readme.md added
Next: figure out what we want the watchdog to do. Then build it and schematic it.
Connections:
- wire segments 63 -> 62
Changed lines of the file:
@@
 L power:GND #PWR?
 U 1 1 5C509E9B
-P 6050 4950
-F 0 "#PWR?" H 6050 4700 50  0001 C CNN
-F 1 "GND" H 6055 4777 50  0000 C CNN
-F 2 "" H 6050 4950 50  0001 C CNN
-F 3 "" H 6050 4950 50  0001 C CNN
-	1    6050 4950
-	1    0    0    -1
+P 6050 4850
+F 0 "#PWR?" H 6050 4600 50  0001 C CNN
+F 1 "GND" H 6055 4677 50  0000 C CNN
+F 2 "" H 6050 4850 50  0001 C CNN
+F 3 "" H 6050 4850 50  0001 C CNN
+	1    6050 4850
+	0    1    1    0
 $EndComp
 Wire Wire Line
 	7300 4750 7550 4750
-Wire Wire Line
-	6050 4950 6050 4850
-Wire Wire Line
-	6050 4850 6150 4850
 Wire Wire Line
 	6250 3950 6250 3900
@@
 Wire Wire Line
 	7150 4750 7250 4750
+Wire Wire Line
+	6050 4850 6150 4850
 $EndSCHEMATC
