File: schematics/motor-and-servo/motor-and-servo.sch (KiCad schematic (older format))
At the start: 6 parts, among them M1 Motor_DC, U1 motor-controller, U2 NRF24L01_Breakout, U3 ThreePinCon

Commit message: Add interrupt connection
Parts:
- removed U3: ThreePinCon, symbol roboamgellan:ThreePinCon
- added U?: three-pin-connector, symbol robomagellan:three-pin-connector
Connections:
- wire segments 56 -> 59
- no-connect marks 1 -> 0
Changed lines of the file:
@@
 Wire Wire Line
 	5350 4100 6000 4100
-NoConn ~ 5150 5700
 Wire Wire Line
 	5150 5400 5400 5400
@@
 Wire Wire Line
 	4650 6100 4650 6000
-$Comp
-L roboamgellan:ThreePinCon U3
-U 1 1 5C50FB3E
-P 7850 3550
-F 0 "U3" H 8077 3351 50  0000 L CNN
-F 1 "ThreePinCon" H 8077 3260 50  0000 L CNN
-F 2 "" H 7850 3550 50  0001 C CNN
-F 3 "" H 7850 3550 50  0001 C CNN
-	1    7850 3550
-	1    0    0    -1
-$EndComp
 Wire Wire Line
 	7000 3800 7700 3800
@@
 Text GLabel 4000 3700 2    50   Input ~ 0
 MotorBattery
+$Comp
+L robomagellan:three-pin-connector U?
+U 1 1 5C5B9FA2
+P 7850 3550
+F 0 "U?" H 8077 3346 50  0000 L CNN
+F 1 "three-pin-connector" H 8077 3255 50  0000 L CNN
+F 2 "" H 7850 3550 50  0001 C CNN
+F 3 "" H 7850 3550 50  0001 C CNN
+	1    7850 3550
+	1    0    0    -1
+$EndComp
+Wire Wire Line
+	5150 5700 5300 5700
+Wire Wire Line
+	5300 5700 5300 3400
+Wire Wire Line
+	5300 3400 6000 3400
 $EndSCHEMATC
